File: Hardware_Desing/LightProyect/LightProyect.kicad_pcb (KiCad board)
At the start: 2 copper layers, 25 x 176 mm, 10 parts, among them J1 Screw_Terminal_01x02, J2 AudioJack2_SwitchT, J3 Screw_Terminal_01x03, M1 Regulator_x_3_3, M2 DC_DC_3_5_module, M3 AudioModule, M4 MPU6050_lite, SW1 SW_Push, U1 ESP-12E

Commit message: PCB desing fixes
Parts:
- moved SW1 24.7 mm to (133.9, 96.2), turned to 90 degrees
- moved J1 24.7 mm to (138.7, 185.8)
- moved J2 24.7 mm to (129.3, 172.6)
- moved M3 24.7 mm to (135.7, 89.1)
- moved M4 24.7 mm to (143.6, 125.1)
- moved D1 24.7 mm to (140.0, 23.8)
- moved M2 24.7 mm to (134.4, 160.4)
- moved J3 24.7 mm to (137.5, 144.7)
- moved M1 24.7 mm to (134.4, 140.1)
- moved U1 23.6 mm to (135.1, 43.3)
Routing:
- net GND: track 195.0 -> 2.29 mm
- net Net-(D1-Pad2): track 31.7 -> 43.2 mm, vias 0 -> 2
- net Net-(SW1-Pad1): track 71.1 -> 62.3 mm
- net Net-(M4-Pad4): track 68.5 -> 75.4 mm, vias 0 -> 1
- net Net-(M1-Pad3): track 87.2 -> 92.7 mm
- net Net-(D1-Pad3): track 175.2 -> 180.2 mm, vias 0 -> 1
- net Net-(M4-Pad3): track 80.7 -> 83.3 mm, vias 0 -> 1
- net Net-(J3-Pad2): track 109.0 -> 111.4 mm
- net Net-(M3-Pad2): track 34.1 -> 35.5 mm, vias 0 -> 1
- net Net-(J3-Pad3): track 102.4 -> 101.1 mm, vias 0 -> 2
- net VCC: track 30.6 -> 29.8 mm
Other:
- board size 25 x 176 mm -> 27 x 176 mm
- board text added: "Designed by Tonix"
- board text added: "Diabolo GDL"

Commit message: Hardware new pcb desing
Parts:
- moved M4 31.3 mm to (112.6, 129.9), turned to 0 degrees
- moved M1 25.2 mm to (122.2, 162.1), turned to 270 degrees
- moved J1 17.6 mm to (121.2, 184.0), turned to 90 degrees
- moved SW1 15.8 mm to (120.6, 104.7)
- moved J3 15.0 mm to (122.5, 145.2)
- moved U1 14.9 mm to (121.8, 50.1)
- moved D1 13.1 mm to (127.9, 29.1)
- moved M3 12.1 mm to (124.6, 93.9)
- moved M2 11.6 mm to (123.2, 157.5)
- moved J2 1.42 mm to (129.6, 174.0), turned to 270 degrees
Connections:
- D1 pad 3: Net-(D1-Pad3) -> Net-(M2-Pad3)
- M1 pad 1: Net-(D1-Pad3) -> Net-(M1-Pad3)
- M1 pad 3: Net-(M1-Pad3) -> Net-(M2-Pad3)
- M2 pad 3: Net-(D1-Pad3) -> Net-(M2-Pad3)
- M2 pad 4: GND -> Net-(M2-Pad4)
- M3 pad 1: Net-(D1-Pad3) -> Net-(M2-Pad3)
Routing:
- net Net-(M2-Pad3): track 0.00 -> 246.6 mm, vias 0 -> 2
- net Net-(D1-Pad3): track 180.2 -> 0.00 mm, vias 1 -> 0
- net Net-(M1-Pad3): track 92.7 -> 125.2 mm, vias 0 -> 2
- net GND: track 2.29 -> 12.4 mm, vias 0 -> 2
- net Net-(M4-Pad4): track 75.4 -> 84.8 mm, vias 1 -> 2
- net Net-(J3-Pad3): track 101.1 -> 94.3 mm, vias 2 -> 0
- net VCC: track 29.8 -> 23.7 mm
- net Net-(J3-Pad2): track 111.4 -> 106.2 mm, vias 0 -> 2
- net Net-(M4-Pad3): track 83.3 -> 80.4 mm, vias 1 -> 2
- net Net-(SW1-Pad1): track 62.3 -> 64.5 mm, vias 0 -> 2
- net Net-(M3-Pad2): track 35.5 -> 34.4 mm, vias 1 -> 0
- net Net-(D1-Pad2): track 43.2 -> 43.9 mm, vias 2 -> 3
- net Net-(M2-Pad4): track 0.00 -> 0.54 mm
Other:
- board size 27 x 176 mm -> 22.9 x 182.2 mm
- rule via_min_size: 0.4 -> 0.2
- board text removed: "Diabolo GDL"

Commit message: Workflow kidCad
Parts:
- removed the D1 at (127.9, 29.1)
- removed the J1 at (121.2, 184.0)
- removed the J2 at (129.6, 174.0)
- removed the J3 at (122.5, 145.2)
- removed the M1 at (122.2, 162.1)
- removed the M2 at (123.2, 157.5)
- removed the M3 at (124.6, 93.9)
- removed the M4 at (112.6, 129.9)
- removed the SW1 at (120.6, 104.7)
- removed the U1 at (121.8, 50.1)
- added D1: NeoPixel_THT, LightProyect:Neopixel, F.Cu at (199.5, 29.5)
- added D1: NeoPixel_THT, LightProyect:Neopixel, F.Cu at (57.8, 29.5)
- added D1: NeoPixel_THT, LightProyect:Neopixel, F.Cu at (92.7, 29.5)
- added D1: NeoPixel_THT, LightProyect:Neopixel, F.Cu at (127.8, 29.3)
- added D1: NeoPixel_THT, LightProyect:Neopixel, F.Cu at (161.8, 28.7)
- added J1: Screw_Terminal_01x02, TerminalBlock:TerminalBlock_bornier-2_P5.08mm, F.Cu at (192.7, 184.4)
- added J1: Screw_Terminal_01x02, TerminalBlock:TerminalBlock_bornier-2_P5.08mm, F.Cu at (51.1, 184.4)
- added J1: Screw_Terminal_01x02, TerminalBlock:TerminalBlock_bornier-2_P5.08mm, F.Cu at (85.9, 184.4)
- added J1: Screw_Terminal_01x02, TerminalBlock:TerminalBlock_bornier-2_P5.08mm, F.Cu at (121.1, 184.1)
- added J1: Screw_Terminal_01x02, TerminalBlock:TerminalBlock_bornier-2_P5.08mm, F.Cu at (155.1, 183.6)
- added J2: AudioJack2_SwitchT, TerminalBlock:TerminalBlock_bornier-3_P5.08mm, F.Cu at (201.2, 174.4)
- added J2: AudioJack2_SwitchT, TerminalBlock:TerminalBlock_bornier-3_P5.08mm, F.Cu at (59.5, 174.4)
- added J2: AudioJack2_SwitchT, TerminalBlock:TerminalBlock_bornier-3_P5.08mm, F.Cu at (94.4, 174.4)
- added J2: AudioJack2_SwitchT, TerminalBlock:TerminalBlock_bornier-3_P5.08mm, F.Cu at (129.5, 174.2)
- added J2: AudioJack2_SwitchT, TerminalBlock:TerminalBlock_bornier-3_P5.08mm, F.Cu at (163.5, 173.6)
- added J3: Screw_Terminal_01x03, TerminalBlock:TerminalBlock_bornier-3_P5.08mm, F.Cu at (194.0, 145.6)
- added J3: Screw_Terminal_01x03, TerminalBlock:TerminalBlock_bornier-3_P5.08mm, F.Cu at (52.4, 145.6)
- added J3: Screw_Terminal_01x03, TerminalBlock:TerminalBlock_bornier-3_P5.08mm, F.Cu at (87.2, 145.6)
- added J3: Screw_Terminal_01x03, TerminalBlock:TerminalBlock_bornier-3_P5.08mm, F.Cu at (122.3, 145.3)
- added J3: Screw_Terminal_01x03, TerminalBlock:TerminalBlock_bornier-3_P5.08mm, F.Cu at (156.3, 144.8)
- added M1: Regulator_x_3_3, LightProyect:YP8AMS1117_5v_3_3_V, F.Cu at (193.7, 162.5)
- added M1: Regulator_x_3_3, LightProyect:YP8AMS1117_5v_3_3_V, F.Cu at (52.1, 162.5)
- added M1: Regulator_x_3_3, LightProyect:YP8AMS1117_5v_3_3_V, F.Cu at (86.9, 162.5)
- added M1: Regulator_x_3_3, LightProyect:YP8AMS1117_5v_3_3_V, F.Cu at (122.0, 162.2)
- added M1: Regulator_x_3_3, LightProyect:YP8AMS1117_5v_3_3_V, F.Cu at (156.0, 161.7)
- added M2: DC_DC_3_5_module, LightProyect:DC_DC_5V_3V_module, F.Cu at (194.7, 157.9)
- added M2: DC_DC_3_5_module, LightProyect:DC_DC_5V_3V_module, F.Cu at (53.1, 157.9)
- added M2: DC_DC_3_5_module, LightProyect:DC_DC_5V_3V_module, F.Cu at (87.9, 157.9)
- added M2: DC_DC_3_5_module, LightProyect:DC_DC_5V_3V_module, F.Cu at (123.0, 157.6)
- added M2: DC_DC_3_5_module, LightProyect:DC_DC_5V_3V_module, F.Cu at (157.0, 157.0)
- added M3: AudioModule, LightProyect:Audio_Senso_module, F.Cu at (195.8, 93.3)
- added M3: AudioModule, LightProyect:Audio_Senso_module, F.Cu at (54.2, 93.3)
- added M3: AudioModule, LightProyect:Audio_Senso_module, F.Cu at (89.0, 93.3)
- added M3: AudioModule, LightProyect:Audio_Senso_module, F.Cu at (124.1, 93.0)
- added M3: AudioModule, LightProyect:Audio_Senso_module, F.Cu at (158.2, 92.4)
- added M4: MPU6050_lite, LightProyect:GY-521, F.Cu at (184.2, 130.3)
- added M4: MPU6050_lite, LightProyect:GY-521, F.Cu at (42.5, 130.3)
- added M4: MPU6050_lite, LightProyect:GY-521, F.Cu at (77.4, 130.3)
- added M4: MPU6050_lite, LightProyect:GY-521, F.Cu at (112.5, 130.0)
- added M4: MPU6050_lite, LightProyect:GY-521, F.Cu at (146.5, 129.4)
- added SW1: SW_Push, Button_Switch_SMD:SW_SPST_TL3305C, F.Cu at (192.1, 105.1)
- added SW1: SW_Push, Button_Switch_SMD:SW_SPST_TL3305C, F.Cu at (50.5, 105.1)
- added SW1: SW_Push, Button_Switch_SMD:SW_SPST_TL3305C, F.Cu at (85.3, 105.1)
- added SW1: SW_Push, Button_Switch_SMD:SW_SPST_TL3305C, F.Cu at (120.4, 104.8)
- added SW1: SW_Push, Button_Switch_SMD:SW_SPST_TL3305C, F.Cu at (154.5, 104.3)
- added U1: ESP-12E, RF_Module:ESP-12E, F.Cu at (193.3, 50.5)
- added U1: ESP-12E, RF_Module:ESP-12E, F.Cu at (51.7, 50.5)
- added U1: ESP-12E, RF_Module:ESP-12E, F.Cu at (86.5, 50.5)
- added U1: ESP-12E, RF_Module:ESP-12E, F.Cu at (121.6, 50.3)
- added U1: ESP-12E, RF_Module:ESP-12E, F.Cu at (155.6, 49.7)
Routing:
- net (no net): track 0.00 -> 2749.8 mm, vias 0 -> 51
- net Net-(M2-Pad3): track 246.6 -> 497.1 mm, vias 2 -> 4
- net Net-(D1-Pad3): track 0.00 -> 250.4 mm, vias 0 -> 4
- net Net-(M1-Pad3): track 125.2 -> 0.00 mm, vias 2 -> 0
- net Net-(J3-Pad2): track 106.2 -> 210.1 mm, vias 2 -> 4
- net Net-(J3-Pad3): track 94.3 -> 188.6 mm
- net Net-(M4-Pad4): track 84.8 -> 169.7 mm, vias 2 -> 4
- net Net-(M4-Pad3): track 80.4 -> 160.9 mm, vias 2 -> 4
- net Net-(SW1-Pad1): track 64.5 -> 129.0 mm, vias 2 -> 4
- net Net-(D1-Pad2): track 43.9 -> 87.9 mm, vias 3 -> 6
- net Net-(M3-Pad2): track 34.4 -> 66.5 mm
- net VCC: track 23.7 -> 47.3 mm
- net GND: track 12.4 -> 24.7 mm, vias 2 -> 4
- net Net-(M2-Pad4): track 0.54 -> 1.07 mm
- added copper zone on F.Cu, net (none)
Other:
- board size 22.9 x 182.2 mm -> 164.5 x 183.1 mm
